File: public/eagle_sch/MCP4725_Breakout.sch (EAGLE design)
At the start: 8 parts, among them U1 DAC_MCP4725SOT-CP

Commit message: download sch
Other:
- note removed: "I2C Address GND = 1100000 (0x60) (Default) VCC - 1100001 (0x61)"
- note removed: "Vcc = 2.7V to 5.5V"
- moved on the sheet: C1, JP6, R1, R2, R3, SJ1, SJ2, U1
Changed lines of the file:
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@@
 <?xml version="1.0" encoding="utf-8"?>
 <!DOCTYPE eagle SYSTEM "eagle.dtd">
-<eagle version="6.1">
+<eagle version="6.4">
 <drawing>
 <settings>
@@
 <part name="SJ2" library="SparkFun-Passives" deviceset="JUMPER-PAD-3-2OF3_NC_BY_PASTE" device="" value=""/>
 <part name="R3" library="SparkFun" deviceset="RESISTOR" device="0603-RES" value="10k"/>
-<part name="FRAME1" library="SparkFun-Aesthetics" deviceset="FRAME-A4L" device=""/>
 </parts>
 <sheets>
 <sheet>
 <plain>
-<text x="63.5" y="7.62" size="1.778" layer="91">I2C Address
-GND = 1100000 (0x60) (Default)
-VCC - 1100001 (0x61)</text>
-<text x="68.58" y="86.36" size="1.778" layer="91">Vcc = 2.7V to 5.5V</text>
 </plain>
 <instances>
-<instance part="C1" gate="G$1" x="109.22" y="45.72"/>
-<instance part="GND1" gate="1" x="109.22" y="38.1"/>
-<instance part="GND5" gate="1" x="40.64" y="40.64"/>
-<instance part="R1" gate="G$1" x="76.2" y="58.42" rot="R90"/>
-<instance part="R2" gate="G$1" x="86.36" y="58.42" rot="R90"/>
-<instance part="P+2" gate="1" x="81.28" y="73.66"/>
-<instance part="P+4" gate="1" x="109.22" y="53.34"/>
-<instance part="P+5" gate="1" x="43.18" y="53.34"/>
-<instance part="U1" gate="G$1" x="58.42" y="48.26"/>
-<instance part="GND2" gate="1" x="53.34" y="22.86"/>
-<instance part="P+1" gate="1" x="81.28" y="33.02"/>
-<instance part="JP6" gate="G$1" x="20.32" y="48.26"/>
-<instance part="SJ1" gate="G$1" x="81.28" y="66.04" rot="R270"/>
-<instance part="SJ2" gate="G$1" x="73.66" y="27.94" rot="R270"/>
-<instance part="R3" gate="G$1" x="60.96" y="27.94"/>
-<instance part="FRAME1" gate="G$1" x="-68.58" y="-40.64"/>
+<instance part="C1" gate="G$1" x="99.06" y="38.1"/>
+<instance part="GND1" gate="1" x="99.06" y="30.48"/>
+<instance part="GND5" gate="1" x="30.48" y="33.02"/>
+<instance part="R1" gate="G$1" x="66.04" y="50.8" rot="R90"/>
+<instance part="R2" gate="G$1" x="76.2" y="50.8" rot="R90"/>
+<instance part="P+2" gate="1" x="71.12" y="66.04"/>
+<instance part="P+4" gate="1" x="99.06" y="45.72"/>
+<instance part="P+5" gate="1" x="33.02" y="45.72"/>
+<instance part="U1" gate="G$1" x="48.26" y="40.64"/>
+<instance part="GND2" gate="1" x="43.18" y="15.24"/>
+<instance part="P+1" gate="1" x="71.12" y="25.4"/>
+<instance part="JP6" gate="G$1" x="10.16" y="40.64"/>
+<instance part="SJ1" gate="G$1" x="71.12" y="58.42" rot="R270"/>
+<instance part="SJ2" gate="G$1" x="63.5" y="20.32" rot="R270"/>
+<instance part="R3" gate="G$1" x="50.8" y="20.32"/>
 </instances>
 <busses>
@@
 <net name="GND" class="0">
 <segment>
-<wire x1="40.64" y1="43.18" x2="40.64" y2="48.26" width="0.1524" layer="91"/>
-<wire x1="40.64" y1="48.26" x2="45.72" y2="48.26" width="0.1524" layer="91"/>
+<wire x1="30.48" y1="35.56" x2="30.48" y2="40.64" width="0.1524" layer="91"/>
+<wire x1="30.48" y1="40.64" x2="35.56" y2="40.64" width="0.1524" layer="91"/>
 <pinref part="GND5" gate="1" pin="GND"/>
 <pinref part="U1" gate="G$1" pin="VSS"/>
 <pinref part="JP6" gate="G$1" pin="1"/>
-<wire x1="27.94" y1="48.26" x2="40.64" y2="48.26" width="0.1524" layer="91"/>
-<junction x="40.64" y="48.26"/>
-</segment>
-<segment>
-<wire x1="109.22" y1="43.18" x2="109.22" y2="40.64" width="0.1524" layer="91"/>
+<wire x1="17.78" y1="40.64" x2="30.48" y2="40.64" width="0.1524" layer="91"/>
+<junction x="30.48" y="40.64"/>
+</segment>
+<segment>
+<wire x1="99.06" y1="35.56" x2="99.06" y2="33.02" width="0.1524" layer="91"/>
 <pinref part="C1" gate="G$1" pin="2"/>
 <pinref part="GND1" gate="1" pin="GND"/>
@@
 <pinref part="R3" gate="G$1" pin="1"/>
 <pinref part="GND2" gate="1" pin="GND"/>
-<wire x1="53.34" y1="25.4" x2="53.34" y2="27.94" width="0.1524" layer="91"/>
-<wire x1="53.34" y1="27.94" x2="55.88" y2="27.94" width="0.1524" layer="91"/>
+<wire x1="43.18" y1="17.78" x2="43.18" y2="20.32" width="0.1524" layer="91"/>
+<wire x1="43.18" y1="20.32" x2="45.72" y2="20.32" width="0.1524" layer="91"/>
 </segment>
 </net>
 <net name="VCC" class="0">
 <segment>
-<wire x1="45.72" y1="45.72" x2="43.18" y2="45.72" width="0.1524" layer="91"/>
-<wire x1="43.18" y1="45.72" x2="43.18" y2="53.34" width="0.1524" layer="91"/>
+<wire x1="35.56" y1="38.1" x2="33.02" y2="38.1" width="0.1524" layer="91"/>
+<wire x1="33.02" y1="38.1" x2="33.02" y2="45.72" width="0.1524" layer="91"/>
 <pinref part="P+5" gate="1" pin="VCC"/>
 <pinref part="U1" gate="G$1" pin="VDD"/>
 </segment>
 <segment>
-<wire x1="109.22" y1="53.34" x2="109.22" y2="50.8" width="0.1524" layer="91"/>
+<wire x1="99.06" y1="45.72" x2="99.06" y2="43.18" width="0.1524" layer="91"/>
 <pinref part="P+4" gate="1" pin="VCC"/>
 <pinref part="C1" gate="G$1" pin="1"/>
@@
 <segment>
 <pinref part="P+2" gate="1" pin="VCC"/>
-<wire x1="81.28" y1="73.66" x2="81.28" y2="71.12" width="0.1524" layer="91"/>
+<wire x1="71.12" y1="66.04" x2="71.12" y2="63.5" width="0.1524" layer="91"/>
 <pinref part="SJ1" gate="G$1" pin="2"/>
 </segment>
 <segment>
 <pinref part="P+1" gate="1" pin="VCC"/>
-<wire x1="78.74" y1="27.94" x2="81.28" y2="27.94" width="0.1524" layer="91"/>
-<wire x1="81.28" y1="27.94" x2="81.28" y2="33.02" width="0.1524" layer="91"/>
+<wire x1="68.58" y1="20.32" x2="71.12" y2="20.32" width="0.1524" layer="91"/>
+<wire x1="71.12" y1="20.32" x2="71.12" y2="25.4" width="0.1524" layer="91"/>
 <pinref part="SJ2" gate="G$1" pin="1"/>
 </segment>
@@
 <net name="SCL" class="0">
 <segment>
-<wire x1="71.12" y1="48.26" x2="76.2" y2="48.26" width="0.1524" layer="91"/>
-<wire x1="76.2" y1="48.26" x2="76.2" y2="53.34" width="0.1524" layer="91"/>
-<wire x1="76.2" y1="48.26" x2="88.9" y2="48.26" width="0.1524" layer="91"/>
-<junction x="76.2" y="48.26"/>
+<wire x1="60.96" y1="40.64" x2="66.04" y2="40.64" width="0.1524" layer="91"/>
+<wire x1="66.04" y1="40.64" x2="66.04" y2="45.72" width="0.1524" layer="91"/>
+<wire x1="66.04" y1="40.64" x2="78.74" y2="40.64" width="0.1524" layer="91"/>
+<junction x="66.04" y="40.64"/>
 <pinref part="R1" gate="G$1" pin="1"/>
-<label x="88.9" y="48.26" size="1.27" layer="95" xref="yes"/>
+<label x="78.74" y="40.64" size="1.27" layer="95" xref="yes"/>
 <pinref part="U1" gate="G$1" pin="SCL"/>
 </segment>
@@
 <net name="SDA" class="0">
 <segment>
-<wire x1="71.12" y1="45.72" x2="86.36" y2="45.72" width="0.1524" layer="91"/>
-<wire x1="86.36" y1="45.72" x2="86.36" y2="53.34" width="0.1524" layer="91"/>
-<wire x1="86.36" y1="45.72" x2="88.9" y2="45.72" width="0.1524" layer="91"/>
-<junction x="86.36" y="45.72"/>
+<wire x1="60.96" y1="38.1" x2="76.2" y2="38.1" width="0.1524" layer="91"/>
+<wire x1="76.2" y1="38.1" x2="76.2" y2="45.72" width="0.1524" layer="91"/>
+<wire x1="76.2" y1="38.1" x2="78.74" y2="38.1" width="0.1524" layer="91"/>
+<junction x="76.2" y="38.1"/>
 <pinref part="R2" gate="G$1" pin="1"/>
-<label x="88.9" y="45.72" size="1.27" layer="95" xref="yes"/>
+<label x="78.74" y="38.1" size="1.27" layer="95" xref="yes"/>
 <pinref part="U1" gate="G$1" pin="SDA"/>
 </segment>
@@
 <segment>
 <pinref part="R2" gate="G$1" pin="2"/>
-<wire x1="86.36" y1="63.5" x2="86.36" y2="66.04" width="0.1524" layer="91"/>
+<wire x1="76.2" y1="55.88" x2="76.2" y2="58.42" width="0.1524" layer="91"/>
 <pinref part="SJ1" gate="G$1" pin="1"/>
 </segment>
@@
 <segment>
 <pinref part="R1" gate="G$1" pin="2"/>
-<wire x1="76.2" y1="63.5" x2="76.2" y2="66.04" width="0.1524" layer="91"/>
+<wire x1="66.04" y1="55.88" x2="66.04" y2="58.42" width="0.1524" layer="91"/>
 <pinref part="SJ1" gate="G$1" pin="3"/>
 </segment>
@@
 <net name="N$3" class="0">
 <segment>
-<wire x1="71.12" y1="50.8" x2="73.66" y2="50.8" width="0.1524" layer="91"/>
-<wire x1="73.66" y1="50.8" x2="73.66" y2="33.02" width="0.1524" layer="91"/>
+<wire x1="60.96" y1="43.18" x2="63.5" y2="43.18" width="0.1524" layer="91"/>
+<wire x1="63.5" y1="43.18" x2="63.5" y2="25.4" width="0.1524" layer="91"/>
 <pinref part="U1" gate="G$1" pin="AO"/>
 <pinref part="SJ2" gate="G$1" pin="2"/>
@@
 <pinref part="U1" gate="G$1" pin="VOUT"/>
 <pinref part="JP6" gate="G$1" pin="2"/>
-<wire x1="45.72" y1="50.8" x2="27.94" y2="50.8" width="0.1524" layer="91"/>
+<wire x1="35.56" y1="43.18" x2="17.78" y2="43.18" width="0.1524" layer="91"/>
 </segment>
 </net>
@@
 <pinref part="SJ2" gate="G$1" pin="3"/>
 <pinref part="R3" gate="G$1" pin="2"/>
-<wire x1="66.04" y1="27.94" x2="68.58" y2="27.94" width="0.1524" layer="91"/>
-</segment>
-</net>
+<wire x1="55.88" y1="20.32" x2="58.42" y2="20.32" width="0.1524" layer="91"/>
+</segment>
+</net>
