File: public/eagle_sch/_TXB0104_breakout_voltage_breakout.sch (EAGLE design)
At the start: 6 parts

Commit message: download sch
Other:
- note removed: "A side Vcc from 1.2 to 3.6V"
- note removed: "B side Vcc from 1.65 to 5V"
- note removed: "VccA *must* be less than VccB!"
- moved on the sheet: C1, C2, JP1, JP2, SJ1, U1
