File: public/eagle_sch/atmega328_5v_16mhz.sch (EAGLE design)
At the start: 9 parts, among them Q1 16MHz, U1 ATMEGA328

Commit message: download sch
Connections:
- net VCC renamed 5V
Other:
- moved on the sheet: C1, C2, C3, D3, Q1, R2, R6, S1, U1
